File: LVDS_LPDDR4_G529/kicad/haasoscope_pro_max/haasoscope_pro_max.kicad_sch (KiCad schematic)
At the start: 4 parts, among them IC1 ADC12DL500ACF, U1 Ti90G529_Functions, U2 MT53E256M32D2DS-046 IT:B, U3 FT601Q

Commit message: Aligned schematics, sort of
Parts:
- removed IC1: ADC12DL500ACF, ADC12DL:BGA256C100P16X16_1700X1700X331, symbol ADC12DL500ACF:ADC12DL500ACF
- removed U1: Ti90G529_Functions, G529:BGA-529_23x23_19.0x19.0mm, symbol Ti90G529_Functions:Ti90G529_Functions
- removed U2: MT53E256M32D2DS-046 IT:B, MT53D512M32D2DS-053 WT_D:IC_MT53D512M16D1DS-046_WT_D, symbol MT53D512M16D1DS:B
- removed U3: FT601Q, Package_DFN_QFN:QFN-76-1EP_9x9mm_P0.4mm_EP5.81x6.31mm, symbol Interface_USB:FT601Q
Other:
- added sheet fpga_config (fpga_config.kicad_sch)
- added sheet fpga_ft601 (fpga_ft601.kicad_sch)
- added sheet fpga_misc (fpga_misc.kicad_sch)
- sheet fpga_ddr: file fpga_adc.kicad_sch -> fpga_ddr.kicad_sch
- sheet fpga_power: file fpga_adc.kicad_sch -> fpga_power.kicad_sch
